Commit message: New example for loading a revolute twins from URDF

File: scs2-examples/src/main/resources/urdf/SimpleRevoluteTwinsRobot.urdf (robot description, URDF)
Before this commit: robot RevoluteTwinsRobot, 2 links, 1 joints
Links:
- link endEffectorLink: geometry visual box size=0.0125 0.0125 0.2
Joints:
- removed joint crossFourBar
- added joint revoluteTwins: type revolute_twins, parent baseLink, child endEffectorLink, axis 0 1 0, limit lower=-1.1 upper=0.4141 effort=190 velocity=5.89
