Commit message: Update mimic to use attributes instead of elements as per URDF spec

File: scs2-examples/src/main/resources/urdf/SimpleRevoluteTwinsRobotTypeC.urdf (robot description, URDF)
Before this commit: robot RevoluteTwinsRobot, 3 links, 3 joints
Joints:
- joint jointB: mimic  -> joint=jointA multiplier=1.25 offset=0
